File: schematic/SAMD21/power.sch (KiCad schematic (older format))
At the start: 34 parts, among them IC2 AZ1117IH-3.3TRG1, J1 Barrel_Jack_Switch, J2 Power, J3 Conn_01x02, J4 Conn_01x02, J5 USB_B_Micro, J6 USB_B_Mini, J7 Conn_01x02, SW1 SW_MEC_5E, SW2 SW_MEC_5E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

Commit message: Complete schematic
Parts:
- C7: footprint Capacitor_SMD:C_0603_1608Metric -> Capacitor_SMD:C_0402_1005Metric
- J5: footprint Connector_USB:USB_Micro-B_Amphenol_10104110_Horizontal -> SamacSys_Parts:USB_Micro-B_Amphenol_10104110_Horizontal-With_pins
Changed lines of the file:
@@
 F 0 "C7" H 4115 4446 50  0000 L CNN
 F 1 "1 uF" H 4115 4355 50  0000 L CNN
-F 2 "Capacitor_SMD:C_0603_1608Metric" H 4038 4250 50  0001 C CNN
+F 2 "Capacitor_SMD:C_0402_1005Metric" H 4038 4250 50  0001 C CNN
 F 3 "~" H 4000 4400 50  0001 C CNN
 	1    4000 4400
@@
 F 0 "J5" H 8370 1389 50  0000 R CNN
 F 1 "USB_B_Micro" H 8370 1298 50  0000 R CNN
-F 2 "Connector_USB:USB_Micro-B_Amphenol_10104110_Horizontal" H 8750 1350 50  0001 C CNN
+F 2 "SamacSys_Parts:USB_Micro-B_Amphenol_10104110_Horizontal-With_pins" H 8750 1350 50  0001 C CNN
 F 3 "~" H 8750 1350 50  0001 C CNN
 	1    8600 1400

Commit message: Moved I2C to pins with support for I2C
Other:
- note added: "VDDIO x 2, VDDIN"
- note removed: "VDDIO x 3"
Changed lines of the file:
@@
 Wire Wire Line
 	2300 4100 2500 4100
-Text Notes 2150 5000 0    50   ~ 0
-VDDIO x 3
+Text Notes 1850 5000 0    50   ~ 0
+VDDIO x 2, VDDIN
 $Comp
 L Device:C C7
@@
 	1    0    0    -1
 $EndComp
-Text GLabel 4650 4250 2    50   Input ~ 0
+Text GLabel 4000 4100 1    50   Input ~ 0
 VDDCORE
 $Comp
@@
 USB_VBUS_SENSE enable
 Wire Wire Line
-	4000 4250 4650 4250
-Wire Wire Line
 	1700 4650 2100 4650
 Text GLabel 1300 6750 0    50   Input ~ 0
@@
 Text GLabel 6200 2250 3    50   Input ~ 0
 PA23
+Wire Wire Line
+	4000 4250 4000 4100
 $EndSCHEMATC

Commit message: Changed LEDs to 0805
Parts:
- D2, D5, D6, D7: footprint LED_SMD:LED_0603_1608Metric -> LED_SMD:LED_0805_2012Metric
Changed lines of the file:
@@
 F 0 "D2" H 7393 4767 50  0000 C CNN
 F 1 "Red" H 7393 4676 50  0000 C CNN
-F 2 "LED_SMD:LED_0603_1608Metric" H 7400 4550 50  0001 C CNN
+F 2 "LED_SMD:LED_0805_2012Metric" H 7400 4550 50  0001 C CNN
 F 3 "~" H 7400 4550 50  0001 C CNN
 	1    7400 4550
@@
 F 0 "D5" H 7793 4767 50  0000 C CNN
 F 1 "Yellow" H 7793 4676 50  0000 C CNN
-F 2 "LED_SMD:LED_0603_1608Metric" H 7800 4550 50  0001 C CNN
+F 2 "LED_SMD:LED_0805_2012Metric" H 7800 4550 50  0001 C CNN
 F 3 "~" H 7800 4550 50  0001 C CNN
 	1    7800 4550
@@
 F 0 "D6" H 8193 4767 50  0000 C CNN
 F 1 "Blue" H 8193 4676 50  0000 C CNN
-F 2 "LED_SMD:LED_0603_1608Metric" H 8200 4550 50  0001 C CNN
+F 2 "LED_SMD:LED_0805_2012Metric" H 8200 4550 50  0001 C CNN
 F 3 "~" H 8200 4550 50  0001 C CNN
 	1    8200 4550
@@
 F 0 "D7" H 8593 4767 50  0000 C CNN
 F 1 "Green" H 8593 4676 50  0000 C CNN
-F 2 "LED_SMD:LED_0603_1608Metric" H 8600 4550 50  0001 C CNN
+F 2 "LED_SMD:LED_0805_2012Metric" H 8600 4550 50  0001 C CNN
 F 3 "~" H 8600 4550 50  0001 C CNN
 	1    8600 4550

Commit message: Changed USB micro footprint
Parts:
- J5: footprint SamacSys_Parts:USB_Micro-B_Amphenol_10104110_Horizontal-With_pins -> Connector_USB:USB_Micro-B_Amphenol_10118194_Horizontal
Changed lines of the file:
@@
 F 0 "J5" H 8370 1389 50  0000 R CNN
 F 1 "USB_B_Micro" H 8370 1298 50  0000 R CNN
-F 2 "SamacSys_Parts:USB_Micro-B_Amphenol_10104110_Horizontal-With_pins" H 8750 1350 50  0001 C CNN
+F 2 "Connector_USB:USB_Micro-B_Amphenol_10118194_Horizontal" H 8750 1350 50  0001 C CNN
 F 3 "~" H 8750 1350 50  0001 C CNN
 	1    8600 1400
